Commit message: feat: lidar ray visualized

File: urdf/attantion.xacro (robot description, xacro)
@@ -1,6 +1,618 @@
 <?xml version="1.0"?>
 <robot xmlns:xacro="http://www.ros.org/wiki/xacro"  name="robot">
-    <xacro:include filename="hunter2_base_gazebo.xacro" />
-    <!-- <xacro:include filename="gazebo_control.xacro" /> -->
-    <xacro:include filename="livox_HAP.xacro" />
+  <link name="base_link">
+    <inertial>
+      <origin
+        xyz="0.0266989327622036 0.000409203500587652 -0.135901124750884"
+        rpy="0 0 0" />
+      <mass
+        value="21.02945169536679" />
+      <inertia
+        ixx="0.0332370959804736"
+        ixy="-1.013150489971E-06"
+        ixz="-0.00188859201421112"
+        iyy="0.111072002332437"
+        iyz="-5.13308150598312E-07"
+        izz="0.12660862809283" />
+    </inertial>
+    <visual>
+      <origin
+        xyz="0 0 0"
+        rpy="0 0 0" />
+      <geometry>
+        <mesh
+          filename="package://hunter2_base/meshes/base_link.STL" />
+      </geometry>
+      <material
+        name="">
+        <color
+          rgba="0.792156862745098 0.819607843137255 0.933333333333333 1" />
+      </material>
+    </visual>
+    <collision>
+      <origin
+        xyz="0 0 0"
+        rpy="0 0 0" />
+      <geometry>
+        <mesh
+          filename="package://hunter2_base/meshes/base_link.STL" />
+      </geometry>
+    </collision>
+  </link>
+  <link
+    name="front_steer_left_link">
+    <inertial>
+      <origin
+        xyz="-0.012614 1.8116E-05 0.0023132"
+        rpy="0 0 0" />
+      <mass
+        value="7.8526" />
+      <inertia
+        ixx="0.063827"
+        ixy="0"
+        ixz="0"
+        iyy="0.063827"
+        iyz="0"
+        izz="0.11091" />
+    </inertial>
+    <visual>
+      <origin
+        xyz="0 0 0"
+        rpy="0 0 0" />
+      <geometry>
+      <cylinder length="0.001" radius="0.005"/>
+      </geometry>
+      <material
+        name="">
+        <color
+          rgba="0.79216 0.81961 0.93333 1" />
+      </material>
+    </visual>
+    <collision>
+      <origin
+        xyz="0 0 0"
+        rpy="0 0 0" />
+      <geometry>
+      <cylinder length="0.001" radius="0.005"/>
+      </geometry>
+    </collision>
+  </link>
+  <joint
+    name="front_steer_left_joint"
+    type="revolute">
+    <origin
+      xyz="0.37142 0.29199 -0.1955"
+      rpy="1.5708 0 0" />
+    <parent
+      link="base_link" />
+    <child
+      link="front_steer_left_link" />
+    <axis
+      xyz="0 1 0" />
+    <limit
+      lower="-0.69"
+      upper="0.69"
+      effort="0"
+      velocity="0" />
+  </joint>
+  <link
+    name="front_left_wheel_link">
+    <inertial>
+      <origin
+        xyz="-6.5774E-06 2.0242E-05 -0.0096386"
+        rpy="0 0 0" />
+      <mass
+        value="7.7007" />
+      <inertia
+        ixx="0.063724"
+        ixy="0"
+        ixz="0"
+        iyy="0.063724"
+        iyz="0"
+        izz="0.11072" />
+    </inertial>
+    <visual>
+      <origin
+        xyz="0 0 0"
+        rpy="0 0 0" />
+      <geometry>
+        <mesh
+          filename="package://hunter2_base/meshes/front_left_wheel_link.STL" />
+      </geometry>
+      <material
+        name="">
+        <color
+          rgba="0.79216 0.81961 0.93333 1" />
+      </material>
+    </visual>
+    <collision>
+      <origin
+        xyz="0 0 0"
+        rpy="0 0 0" />
+      <geometry>
+        <mesh
+          filename="package://hunter2_base/meshes/front_left_wheel_link.STL" />
+      </geometry>
+    </collision>
+  </link>
+  <joint
+    name="front_left_wheel_joint"
+    type="continuous">
+    <origin
+      xyz="0 0 0"
+      rpy="0 0 0" />
+    <parent
+      link="front_steer_left_link" />
+    <child
+      link="front_left_wheel_link" />
+    <axis
+      xyz="0 0 -1" />
+      <dynamics damping="0.0" friction="15"/>
+  </joint>
+  <link
+    name="front_steer_right_link">
+    <inertial>
+      <origin
+        xyz="-8.9374E-08 1.0997E-07 0.0095958"
+        rpy="0 0 0" />
+      <mass
+        value="7.696" />
+      <inertia
+        ixx="0.063704"
+        ixy="0"
+        ixz="0"
+        iyy="0.063704"
+        iyz="0"
+        izz="0.11068" />
+    </inertial>
+    <visual>
+      <origin
+        xyz="0 0 0"
+        rpy="0 0 0" />
+      <geometry>
+      <cylinder length="0.001" radius="0.005"/>
+      </geometry>
+      <material
+        name="">
+        <color
+          rgba="0.79216 0.81961 0.93333 1" />
+      </material>
+    </visual>
+    <collision>
+      <origin
+        xyz="0 0 0"
+        rpy="0 0 0" />
+      <geometry>
+      <cylinder length="0.001" radius="0.005"/>
+      </geometry>
+    </collision>
+  </link>
+  <joint
+    name="front_steer_right_joint"
+    type="revolute">
+    <origin
+      xyz="0.37142 -0.29201 -0.1955"
+      rpy="1.5708 0 0" />
+    <parent
+      link="base_link" />
+    <child
+      link="front_steer_right_link" />
+    <axis
+      xyz="0 1 0" />
+    <limit
+      lower="-0.69"
+      upper="0.69"
+      effort="0"
+      velocity="0" />
+  </joint>
+  <link
+    name="front_right_wheel_link">
+    <inertial>
+      <origin
+        xyz="-9.1148E-08 1.1284E-07 0.0095049"
+        rpy="0 0 0" />
+      <mass
+        value="7.5613" />
+      <inertia
+        ixx="0.063626"
+        ixy="0"
+        ixz="0"
+        iyy="0.063626"
+        iyz="0"
+        izz="0.11054" />
+    </inertial>
+    <visual>
+      <origin
+        xyz="0 0 0"
+        rpy="0 3.14 0" />
+      <geometry>
+        <mesh
+          filename="package://hunter2_base/meshes/front_left_wheel_link.STL" />
+      </geometry>
+      <material
+        name="">
+        <color
+          rgba="0.79216 0.81961 0.93333 1" />
+      </material>
+    </visual>
+    <collision>
+      <origin
+        xyz="0 0 0"
+        rpy="0 0 0" />
+      <geometry>
+        <mesh
+          filename="package://hunter2_base/meshes/front_right_wheel_link.STL" />
+      </geometry>
+    </collision>
+  </link>
+  <joint
+    name="front_right_wheel_joint"
+    type="continuous">
+    <origin
+      xyz="0 0 0"
+      rpy="0 0 0" />
+    <parent
+      link="front_steer_right_link" />
+    <child
+      link="front_right_wheel_link" />
+    <axis
+      xyz="0 0 -1" />
+      <dynamics damping="0.0" friction="15"/>
+  </joint>
+  <link
+    name="left_rear_link">
+    <inertial>
+      <origin
+        xyz="-8.826E-05 6.4342E-05 -0.0096491"
+        rpy="0 0 0" />
+      <mass
+        value="7.6692" />
+      <inertia
+        ixx="0.063699"
+        ixy="0"
+        ixz="0"
+        iyy="0.063699"
+        iyz="0"
+        izz="0.11067" />
+    </inertial>
+    <visual>
+      <origin
+        xyz="0 0 0"
+        rpy="0 0 0" />
+      <geometry>
+        <mesh
+          filename="package://hunter2_base/meshes/left_rear_link.STL" />
+      </geometry>
+      <material
+        name="">
+        <color
+          rgba="0.79216 0.81961 0.93333 1" />
+      </material>
+    </visual>
+    <collision>
+      <origin
+        xyz="0 0 0"
+        rpy="0 0 0" />
+      <geometry>
+        <mesh
+          filename="package://hunter2_base/meshes/left_rear_link.STL" />
+      </geometry>
+    </collision>
+  </link>
+  <joint
+    name="left_rear_joint"
+    type="continuous">
+    <origin
+      xyz="-0.28 0.29249 -0.19558"
+      rpy="1.5708 0 0" />
+    <parent
+      link="base_link" />
+    <child
+      link="left_rear_link" />
+    <axis
+      xyz="0 0 -1" />
+     <dynamics damping="0.0" friction="15"/>
+  </joint>
+  <link
+    name="right_rear_link">
+    <inertial>
+      <origin
+        xyz="8.6344E-05 7.4488E-05 0.0097824"
+        rpy="0 0 0" />
+      <mass
+        value="7.7133" />
+      <inertia
+        ixx="0.06373"
+        ixy="0"
+        ixz="0"
+        iyy="0.06373"
+        iyz="0"
+        izz="0.11073" />
+    </inertial>
+    <visual>
+      <origin
+        xyz="0 0 0"
+        rpy="0 0 0" />
+      <geometry>
+        <mesh
+          filename="package://hunter2_base/meshes/right_rear_link.STL" />
+      </geometry>
+      <material
+        name="">
+        <color
+          rgba="0.79216 0.81961 0.93333 1" />
+      </material>
+    </visual>
+    <collision>
+      <origin
+        xyz="0 0 0"
+        rpy="0 0 0" />
+      <geometry>
+        <mesh
+          filename="package://hunter2_base/meshes/right_rear_link.STL" />
+      </geometry>
+    </collision>
+  </link>
+  <joint
+    name="right_rear_joint"
+    type="continuous">
+    <origin
+      xyz="-0.28018 -0.29251 -0.19558"
+      rpy="1.5708 0.0026575 0" />
+    <parent
+      link="base_link" />
+    <child
+      link="right_rear_link" />
+    <axis
+      xyz="0 0 -1" />
+     <dynamics damping="0.0" friction="15"/>
+  </joint>
+  <link
+    name="front_steer_link">
+    <inertial>
+      <origin
+        xyz="0.049836 8.1046E-15 0.017912"
+        rpy="0 0 0" />
+      <mass
+        value="0.0049179" />
+      <inertia
+        ixx="1.6846E-07"
+        ixy="7.6396E-23"
+        ixz="-1.0974E-08"
+        iyy="7.549E-07"
+        iyz="-1.8957E-22"
+        izz="7.334E-07" />
+    </inertial>
+    <visual>
+      <origin
+        xyz="0 0 0"
+        rpy="0 0 0" />
+      <geometry>
+      <cylinder length="0.001" radius="0.005"/>
+      </geometry>
+      <material
+        name="">
+        <color
+          rgba="0.79216 0.81961 0.93333 1" />
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
File: urdf/livox_HAP.xacro (robot description, xacro)
@@ -1,8 +1,10 @@
-<?xml version="1.0" encoding="utf-8"?>
-<!-- This URDF was automatically created by SolidWorks to URDF Exporter! Originally created by Stephen Brawner (brawner@gmail.com)
-     Commit Version: 1.6.0-1-g15f4949  Build Version: 1.6.7594.29634
-     For more information, please see http://wiki.ros.org/sw_urdf_exporter -->
-<robot xmlns:xacro = "http://www.ros.org.wiki/xacro">
-  <!-- start here to *  -->
+<?xml version="1.0"?>
+<robot xmlns:xacro="http://ros.org/wiki/xacro">
+  <xacro:property name="M_PI" value="3.14159"/>
+  <xacro:property name="laser_min_range" value="0.1"/>
+  <xacro:property name="laser_max_range" value="200.0"/>
+  <xacro:property name="ros_topic" value="scan"/>
+  <xacro:property name="samples" value="45300"/>
+  <xacro:property name="downsample" value="0"/>
   <xacro:macro name="null_inertial">
     <inertial>
@@ -13,74 +15,74 @@
     </inertial>
   </xacro:macro>
-  <xacro:macro name="Livox_Hap_gazebo" params="name:=livox_HAP">
-    <gazebo reference="livox_HAP">
-      <sensor type="ray" name="laser_livox_HAP">
+  <xacro:macro name="Livox_Mid_gazebo_sensor" params="visualize:=True update_rate:=10 resolution:=0.002 noise_mean:=0.0 noise_stddev:=0.01 name:=livox">
+    <gazebo reference="${name}">
+      <sensor type="ray" name="laser_${name}">
         <pose>0 0 0 0 0 0</pose>
-        <visualize>true</visualize>
-        <update_rate>10</update_rate>
+        <visualize>${visualize}</visualize>
+        <update_rate>${update_rate}</update_rate>
         <!-- This ray plgin is only for visualization. -->
         <plugin name="gazebo_ros_laser_controller" filename="liblivox_laser_simulation.so">
-			  <ray>
-          <scan>
-            <horizontal>
-              <samples>100</samples>
-              <resolution>1</resolution>
-		    		  <min_angle>-1.047196667</min_angle>
-		    		  <max_angle>1.047196667</max_angle>
-            </horizontal>
-            <vertical>
-		    		  <samples>50</samples>
-		    		  <resolution>1</resolution>
-		    		  <min_angle>-0.218165972</min_angle>
-		    		  <max_angle>0.218165972</max_angle>
-		    		</vertical>
-          </scan>
-          <range>
-		    		<min>0.1</min>
-		    		<max>200.0</max>
-		    		<resolution>0.002</resolution>
-          </range>
-          <noise>
-		    		<type>gaussian</type>
-		    		<mean>0.0</mean>
-		    		<stddev>0.01</stddev>
-		    	</noise>
-        </ray>
+      <ray>
+			  <scan>
+				<horizontal>
+				<samples>100</samples>
+				<resolution>1</resolution>
+				<min_angle>${-60/180*M_PI}</min_angle>
+				<max_angle>${60/180*M_PI}</max_angle>
+				</horizontal>
+				<vertical>
+				<samples>50</samples>
+				<resolution>1</resolution>
+				<min_angle>${-12.5/180*M_PI}</min_angle>
+				<max_angle>${12.5/180*M_PI}</max_angle>
+				</vertical>
+			  </scan>
+			  <range>
+				<min>${laser_min_range}</min>
+				<max>${laser_max_range}</max>
+				<resolution>${resolution}</resolution>
+			  </range>
+			  <noise>
+				<type>gaussian</type>
+				<mean>${noise_mean}</mean>
+				<stddev>${noise_stddev}</stddev>
+			  </noise>
+			</ray>
       <visualize>true</visualize>
-		  <samples>45300</samples>
+		  <samples>${samples}</samples>
 		  <downsample>1</downsample>
-		  <csv_file_name>package://immersion_sim/scan_mode/HAP.csv</csv_file_name>
-		  <ros_topic>scan</ros_topic>
-      </plugin>
+		  <!-- <csv_file_name>package://immersion_sim/scan_mode/HAP.csv</csv_file_name> -->
+		  <ros_topic>${ros_topic}</ros_topic>
+        </plugin>
       </sensor>
     </gazebo>
   </xacro:macro>
-  <xacro:macro name="Livox_HAP" params="visualize:=True name:=livox">
-    <link name="Livox_HAP_base">
+  <xacro:macro name="Livox_Mid40" params="visualize:=True name:=livox">
+    <link name="lidar_base">
       <xacro:null_inertial/>
       <visual>
-        <origin xyz="0.0 0.0 0.0" rpy="0 0 0"/>
+        <origin xyz="0.00 0 0.0" rpy="0 0 0"/>
         <geometry>
-          <mesh filename="package://immersion_sim/meshes/livox_mid40.dae">
+          <mesh filename="package://livox_laser_simulation/meshes/livox_mid40.dae">
           </mesh>
         </geometry>
       </visual>
       <collision>
-		    <origin xyz="0.0 0.0 0.0" rpy="0 0 0" /> <geometry>
-        <mesh filename="package://immersion_sim/meshes/livox_mid40.dae"> </mesh>
-        </geometry>
+		  <origin xyz="0 0 0" rpy="0 0 0" /> <geometry>
+        <mesh filename="package://livox_laser_simulation/meshes/livox_mid40.dae"> </mesh>
+      </geometry>
       </collision>
     </link>
-    <link name="Livox_HAP">
+    <link name="lidar">
       <xacro:null_inertial/>
     </link>
-    <joint name="Livox_HAP_base_to_Livox_HAP_joint" type="fixed">
-      <parent link="Livox_HAP_base"/>
-      <child link="Livox_HAP"/>
-      <origin xyz="0.0 0.0 0.0" rpy="0 0 0" />
+    <joint name="lidar_to_lidar_base_joint" type="fixed">
+      <parent link="lidar_base"/>
+      <child link="lidar"/>
+      <origin rpy="0 0 0" xyz="0.0 0.0 1.6"/>
     </joint>
-    <xacro:Livox_Hap_gazebo name="livox_HAP"/>
+    <xacro:Livox_Mid_gazebo_sensor name="lidar" visualize="true"/>
   </xacro:macro>
-  <xacro:Livox_HAP name="livox_HAP"/>
+  <xacro:Livox_Mid40 name="hap"/>
   <joint name="base_link_to_lidar_joint" type="fixed">
     <origin xyz="0.0 0.0 0.5" rpy="0.0 0.0 1.58"/>

Commit message: feat: /scan topic publish

File: urdf/attantion.xacro (robot description, xacro)
@@ -534,39 +534,41 @@
       <sensor type="ray" name="laser_${name}">
         <pose>0 0 0 0 0 0</pose>
-        <visualize>${visualize}</visualize>
-        <update_rate>${update_rate}</update_rate>
-        <!-- This ray plgin is only for visualization. -->
-        <!-- <plugin name="gazebo_ros_laser_controller" filename="liblivox_laser_simulation.so"> -->
-		<ray>
-		  <scan>
-			<horizontal>
-			<samples>100</samples>
-			<resolution>1</resolution>
-			<min_angle>${-60/180*M_PI}</min_angle>
-			<max_angle>${60/180*M_PI}</max_angle>
-			</horizontal>
-			<vertical>
-			<samples>50</samples>
-			<resolution>1</resolution>
-			<min_angle>${-12.5/180*M_PI}</min_angle>
-			<max_angle>${12.5/180*M_PI}</max_angle>
-			</vertical>
-		  </scan>
-		  <range>
-			<min>${laser_min_range}</min>
-			<max>${laser_max_range}</max>
-			<resolution>${resolution}</resolution>
-		  </range>
-		  <noise>
-			<type>gaussian</type>
-			<mean>${noise_mean}</mean>
-			<stddev>${noise_stddev}</stddev>
-		  </noise>
-		</ray>
-        <visualize>${visualize}</visualize>
-		<samples>${samples}</samples>
-		<downsample>${downsample}</downsample>
-		<csv_file_name>package://livox_laser_simulation/scan_mode/HAP.csv</csv_file_name>
-		<ros_topic>${ros_topic}</ros_topic>
+        <visualize>true</visualize>
+        <update_rate>10</update_rate>
+        <!-- <plugin name="lidar_plugin" filename="libgazebo_ros_pointcloud.so"> -->
+        <!-- <frameName>lidar</frameName> -->
+		    <ray>
+		      <scan>
+		    	<horizontal>
+		    	<samples>100</samples>
+		    	<resolution>1</resolution>
+		    	<min_angle>${-60/180*M_PI}</min_angle>
+		    	<max_angle>${60/180*M_PI}</max_angle>
+		    	</horizontal>
+		    	<vertical>
+		    	<samples>50</samples>
+		    	<resolution>1</resolution>
+		    	<min_angle>${-12.5/180*M_PI}</min_angle>
+		    	<max_angle>${12.5/180*M_PI}</max_angle>
+		    	</vertical>
+		      </scan>
+		      <range>
+		    	<min>${laser_min_range}</min>
+		    	<max>${laser_max_range}</max>
+		    	<resolution>${resolution}</resolution>
+		      </range>
+		      <noise>
+		    	<type>gaussian</type>
+		    	<mean>${noise_mean}</mean>
+		    	<stddev>${noise_stddev}</stddev>
+		      </noise>
+		    </ray>
+        <plugin name="BLS_1_link_controller" filename="libgazebo_ros_block_laser.so">
+        <topicName>/scan</topicName>
+        <frameName>lidar</frameName>
+        </plugin>
+		    <samples>${samples}</samples>
+		    <downsample>${downsample}</downsample>
+		    <!-- <topicName>/scan</topicName> -->
         <!-- </plugin> -->
       </sensor>
@@ -601,5 +603,5 @@
   <xacro:Livox_Mid40 name="hap"/>
   <joint name="base_link_to_lidar_joint" type="fixed">
-      <origin xyz="0.0 0.0 0.5" rpy="0.0 0.0 1.58"/>
+      <origin xyz="0.0 0.0 0.5" rpy="0.0 0.0 0.0"/>
       <parent link="base_link"/>
       <child link="lidar_base"/>

Commit message: feat: update for HAP lidar

File: urdf/attantion.xacro (robot description, xacro)
@@ -538,5 +538,12 @@
         <!-- <plugin name="lidar_plugin" filename="libgazebo_ros_pointcloud.so"> -->
         <!-- <frameName>lidar</frameName> -->
-		    <ray>
+        <plugin name="gazebo_ros_laser_controller" filename="liblivox_laser_simulation.so">
+          <frameName>lidar</frameName>
+          <visualize>true</visualize>
+		      <samples>${samples}</samples>
+		      <downsample>1</downsample>
+		      <csv_file_name>package://immersion_sim/scan_mode/HAP.csv</csv_file_name>
+		      <ros_topic>scan</ros_topic>
+          <ray>
 		      <scan>
 		    	<horizontal>
@@ -564,7 +571,4 @@
 		      </noise>
 		    </ray>
-        <plugin name="BLS_1_link_controller" filename="libgazebo_ros_block_laser.so">
-        <topicName>/scan</topicName>
-        <frameName>lidar</frameName>
         </plugin>
 		    <samples>${samples}</samples>
@@ -595,5 +599,5 @@
     </link>
     <joint name="lidar_to_lidar_base_joint" type="fixed">
-      <parent link="lidar_base"/>
+      <parent link="base_link"/>
       <child link="lidar"/>
       <origin rpy="0 0 0" xyz="0.0 0.0 0.0"/>

File: urdf/livox_HAP.xacro (robot description, xacro)
@@ -52,5 +52,5 @@
 		  <samples>${samples}</samples>
 		  <downsample>1</downsample>
-		  <!-- <csv_file_name>package://immersion_sim/scan_mode/HAP.csv</csv_file_name> -->
+		  <csv_file_name>package://immersion_sim/scan_mode/HAP.csv</csv_file_name>
 		  <ros_topic>${ros_topic}</ros_topic>
         </plugin>

Commit message: feat: tf base_link

File: urdf/attantion.xacro (robot description, xacro)
@@ -531,13 +531,11 @@
   </xacro:macro>
   <xacro:macro name="Livox_Mid_gazebo_sensor" params="visualize:=True update_rate:=10 resolution:=0.002 noise_mean:=0.0 noise_stddev:=0.01 name:=livox">
-    <gazebo reference = "${name}">
-      <sensor type="ray" name="laser_${name}">
+    <gazebo reference="${name}">
+      <sensor type="ray" name="${name}">
         <pose>0 0 0 0 0 0</pose>
         <visualize>true</visualize>
         <update_rate>10</update_rate>
-        <!-- <plugin name="lidar_plugin" filename="libgazebo_ros_pointcloud.so"> -->
-        <!-- <frameName>lidar</frameName> -->
         <plugin name="gazebo_ros_laser_controller" filename="liblivox_laser_simulation.so">
-          <frameName>lidar</frameName>
+          <!-- <frameName>lidar</frameName> -->
           <visualize>true</visualize>
 		      <samples>${samples}</samples>
@@ -572,16 +570,12 @@
 		    </ray>
         </plugin>
-		    <samples>${samples}</samples>
-		    <downsample>${downsample}</downsample>
-		    <!-- <topicName>/scan</topicName> -->
-        <!-- </plugin> -->
       </sensor>
     </gazebo>
   </xacro:macro>
   <xacro:macro name="Livox_Mid40" params="visualize:=True name:=livox">
-    <link name="lidar_base">
+    <link name="lidar">
       <xacro:null_inertial/>
       <visual>
-        <origin xyz="0.00 0 1.0" rpy="0 0 0"/>
+        <origin xyz="0.00 0 0.0" rpy="0 0 0"/>
         <geometry>
           <mesh filename="package://livox_laser_simulation/meshes/livox_mid40.dae">
@@ -595,12 +589,4 @@
       </collision>
     </link>
-    <link name="lidar">
-      <xacro:null_inertial/>
-    </link>
-    <joint name="lidar_to_lidar_base_joint" type="fixed">
-      <parent link="base_link"/>
-      <child link="lidar"/>
-      <origin rpy="0 0 0" xyz="0.0 0.0 0.0"/>
-    </joint>
     <xacro:Livox_Mid_gazebo_sensor name="lidar" visualize="true"/>
   </xacro:macro>
@@ -609,5 +595,5 @@
       <origin xyz="0.0 0.0 0.5" rpy="0.0 0.0 0.0"/>
       <parent link="base_link"/>
-      <child link="lidar_base"/>
+      <child link="lidar"/>
   </joint>
   <gazebo>
@@ -616,9 +602,4 @@
       <legacyModeNS>false</legacyModeNS>
     </plugin>
-    <!-- <joint name="base_link_to_lidar_joint" type="fixed">
-        <parent>base_link</parent>
-        <child>lidar_base</child>
-        <pose>0.0 0.0 0.5 0.0 0.0 1.58</pose>
-    </joint> -->
   </gazebo>
 </robot>
